Commit message: update g1 23-DOF hip_pitch to mode 10 values (effort 139, velocity 20)

File: src/holosoma/holosoma/data/robots/g1/g1_23dof.urdf (robot description, URDF)
Before this commit: robot g1_23dof, 34 links, 33 joints
Joints:
- joint left_hip_pitch_joint: limit lower=-2.5307 upper=2.8798 effort=88 velocity=32 -> lower=-2.5307 upper=2.8798 effort=139 velocity=20
- joint right_hip_pitch_joint: limit lower=-2.5307 upper=2.8798 effort=88 velocity=32 -> lower=-2.5307 upper=2.8798 effort=139 velocity=20
